File: PCB files/ece196LiDAR/ece196LiDAR.kicad_sch (KiCad schematic)
At the start: 8 parts, among them J1 Conn_01x20_Pin, J2 Conn_01x20_Pin, J3 Conn_01x05_Pin, J4 Conn_01x05_Pin, J5 Conn_01x05_Pin, J6 Conn_01x05_Pin, J7 Conn_01x05_Pin, J8 Conn_01x02_Pin

Commit message: PCB submission
Parts:
- added D1: LED, symbol Device:LED
- added R1: R, symbol Device:R
Connections:
- net +5V: now also R1.1
- net GND: now also D1.1 (K)
- new net: D1.2 (A), R1.2
Other:
- note added: "global label BAD"
